File: pruebakicad/prueba.kicad_pcb (KiCad board)
At the start: 2 copper layers, 33 parts, among them J1 Conn_01x08_RC522, J2 Conn_01x04_MountingPin, J3 Conn_01x03, J4 Conn_2Rows-15Pins, J5 Conn_01x04, Q1 BSS138, Q2 BSS138, U1 TLV1117-33, U2 TLV1117-50, U3 ESP32-WROOM-32

Commit message: wires
Parts:
- added R2: 0R, Resistor_SMD:R_0805_2012Metric, F.Cu at (78.7, 106.7)
- added R6: 0R, Resistor_SMD:R_0805_2012Metric, F.Cu at (78.7, 109.6)
- added R7: 0R, Resistor_SMD:R_0805_2012Metric, F.Cu at (83.2, 106.7)
- moved R4 19.0 mm to (72.4, 102.9)
- moved C2 18.1 mm to (67.3, 99.1), turned to 180 degrees
- moved R1 12.3 mm to (72.0, 106.7)
- moved SWBOOTesp1 11.7 mm to (73.5, 87.6)
- moved Q1 11.0 mm to (77.2, 100.0), turned to 180 degrees
- moved C3 3.81 mm to (67.3, 106.7)
- moved C5 3.81 mm to (66.8, 102.9)
Changed lines of the file:
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@@
     (tracks 0)
     (zones 0)
-    (modules 33)
+    (modules 36)
     (nets 48)
   )
@@
     (add_net "Net-(U3-Pad32)")
   )
+  (module Resistor_SMD:R_0805_2012Metric (layer F.Cu)
+    (at 83.15 106.68)
+    (descr "Resistor SMD 0805 (2012 Metric), square (rectangular) end terminal, IPC_7351 nominal, (Body size source: IPC-SM-782 page 72, https://www.pcb-3d.com/wordpress/wp-content/uploads/ipc-sm-782a_amendment_1_and_2.pdf), generated with kicad-footprint-generator")
+    (tags resistor)
+    (attr smd)
+    (fp_text reference R7 (at 0 -1.65) (layer F.SilkS)
+      (effects (font (size 1 1) (thickness 0.15)))
+    )
+    (fp_text value 0R (at 0 1.65) (layer F.Fab)
+      (effects (font (size 1 1) (thickness 0.15)))
+    )
+    (fp_text user %R (at 0 0) (layer F.Fab)
+      (effects (font (size 0.5 0.5) (thickness 0.08)))
+    )
+    (fp_line (start -1 0.625) (end -1 -0.625) (layer F.Fab) (width 0.1))
+    (fp_line (start -1 -0.625) (end 1 -0.625) (layer F.Fab) (width 0.1))
+    (fp_line (start 1 -0.625) (end 1 0.625) (layer F.Fab) (width 0.1))
+    (fp_line (start 1 0.625) (end -1 0.625) (layer F.Fab) (width 0.1))
+    (fp_line (start -0.227064 -0.735) (end 0.227064 -0.735) (layer F.SilkS) (width 0.12))
+    (fp_line (start -0.227064 0.735) (end 0.227064 0.735) (layer F.SilkS) (width 0.12))
+    (fp_line (start -1.68 0.95) (end -1.68 -0.95) (layer F.CrtYd) (width 0.05))
+    (fp_line (start -1.68 -0.95) (end 1.68 -0.95) (layer F.CrtYd) (width 0.05))
+    (fp_line (start 1.68 -0.95) (end 1.68 0.95) (layer F.CrtYd) (width 0.05))
+    (fp_line (start 1.68 0.95) (end -1.68 0.95) (layer F.CrtYd) (width 0.05))
+    (pad 2 smd roundrect (at 0.9125 0) (size 1.025 1.4) (layers F.Cu F.Paste F.Mask) (roundrect_rratio 0.243902)
+      (net 38 "Net-(Q2-Pad3)"))
+    (pad 1 smd roundrect (at -0.9125 0) (size 1.025 1.4) (layers F.Cu F.Paste F.Mask) (roundrect_rratio 0.243902)
+      (net 45 /esp32-wroom/IO2))
+    (model ${KISYS3DMOD}/Resistor_SMD.3dshapes/R_0805_2012Metric.wrl
+      (at (xyz 0 0 0))
+      (scale (xyz 1 1 1))
+      (rotate (xyz 0 0 0))
+    )
+  )
+  (module Resistor_SMD:R_0805_2012Metric (layer F.Cu)
+    (at 78.74 109.63)
+    (descr "Resistor SMD 0805 (2012 Metric), square (rectangular) end terminal, IPC_7351 nominal, (Body size source: IPC-SM-782 page 72, https://www.pcb-3d.com/wordpress/wp-content/uploads/ipc-sm-782a_amendment_1_and_2.pdf), generated with kicad-footprint-generator")
+    (tags resistor)
+    (attr smd)
+    (fp_text reference R6 (at 0 -1.65) (layer F.SilkS)
+      (effects (font (size 1 1) (thickness 0.15)))
+    )
+    (fp_text value 0R (at 0 1.65) (layer F.Fab)
+      (effects (font (size 1 1) (thickness 0.15)))
+    )
+    (fp_text user %R (at 0 0) (layer F.Fab)
+      (effects (font (size 0.5 0.5) (thickness 0.08)))
+    )
+    (fp_line (start -1 0.625) (end -1 -0.625) (layer F.Fab) (width 0.1))
+    (fp_line (start -1 -0.625) (end 1 -0.625) (layer F.Fab) (width 0.1))
+    (fp_line (start 1 -0.625) (end 1 0.625) (layer F.Fab) (width 0.1))
+    (fp_line (start 1 0.625) (end -1 0.625) (layer F.Fab) (width 0.1))
+    (fp_line (start -0.227064 -0.735) (end 0.227064 -0.735) (layer F.SilkS) (width 0.12))
+    (fp_line (start -0.227064 0.735) (end 0.227064 0.735) (layer F.SilkS) (width 0.12))
+    (fp_line (start -1.68 0.95) (end -1.68 -0.95) (layer F.CrtYd) (width 0.05))
+    (fp_line (start -1.68 -0.95) (end 1.68 -0.95) (layer F.CrtYd) (width 0.05))
+    (fp_line (start 1.68 -0.95) (end 1.68 0.95) (layer F.CrtYd) (width 0.05))
+    (fp_line (start 1.68 0.95) (end -1.68 0.95) (layer F.CrtYd) (width 0.05))
+    (pad 2 smd roundrect (at 0.9125 0) (size 1.025 1.4) (layers F.Cu F.Paste F.Mask) (roundrect_rratio 0.243902)
+      (net 35 "Net-(Q1-Pad3)"))
+    (pad 1 smd roundrect (at -0.9125 0) (size 1.025 1.4) (layers F.Cu F.Paste F.Mask) (roundrect_rratio 0.243902)
+      (net 46 /esp32-wroom/IO0))
+    (model ${KISYS3DMOD}/Resistor_SMD.3dshapes/R_0805_2012Metric.wrl
+      (at (xyz 0 0 0))
+      (scale (xyz 1 1 1))
+      (rotate (xyz 0 0 0))
+    )
+  )
+  (module Resistor_SMD:R_0805_2012Metric (layer F.Cu)
+    (at 78.74 106.68)
+    (descr "Resistor SMD 0805 (2012 Metric), square (rectangular) end terminal, IPC_7351 nominal, (Body size source: IPC-SM-782 page 72, https://www.pcb-3d.com/wordpress/wp-content/uploads/ipc-sm-782a_amendment_1_and_2.pdf), generated with kicad-footprint-generator")
+    (tags resistor)
+    (attr smd)
+    (fp_text reference R2 (at 0 -1.65) (layer F.SilkS)
+      (effects (font (size 1 1) (thickness 0.15)))
+    )
+    (fp_text value 0R (at 0 1.65) (layer F.Fab)
+      (effects (font (size 1 1) (thickness 0.15)))
+    )
+    (fp_text user %R (at 0 0) (layer F.Fab)
+      (effects (font (size 0.5 0.5) (thickness 0.08)))
+    )
+    (fp_line (start -1 0.625) (end -1 -0.625) (layer F.Fab) (width 0.1))
+    (fp_line (start -1 -0.625) (end 1 -0.625) (layer F.Fab) (width 0.1))
+    (fp_line (start 1 -0.625) (end 1 0.625) (layer F.Fab) (width 0.1))
+    (fp_line (start 1 0.625) (end -1 0.625) (layer F.Fab) (width 0.1))
+    (fp_line (start -0.227064 -0.735) (end 0.227064 -0.735) (layer F.SilkS) (width 0.12))
+    (fp_line (start -0.227064 0.735) (end 0.227064 0.735) (layer F.SilkS) (width 0.12))
+    (fp_line (start -1.68 0.95) (end -1.68 -0.95) (layer F.CrtYd) (width 0.05))
+    (fp_line (start -1.68 -0.95) (end 1.68 -0.95) (layer F.CrtYd) (width 0.05))
+    (fp_line (start 1.68 -0.95) (end 1.68 0.95) (layer F.CrtYd) (width 0.05))
+    (fp_line (start 1.68 0.95) (end -1.68 0.95) (layer F.CrtYd) (width 0.05))
+    (pad 2 smd roundrect (at 0.9125 0) (size 1.025 1.4) (layers F.Cu F.Paste F.Mask) (roundrect_rratio 0.243902)
+      (net 7 "Net-(C4-Pad1)"))
+    (pad 1 smd roundrect (at -0.9125 0) (size 1.025 1.4) (layers F.Cu F.Paste F.Mask) (roundrect_rratio 0.243902)
+      (net 6 /esp32-wroom/EN))
+    (model ${KISYS3DMOD}/Resistor_SMD.3dshapes/R_0805_2012Metric.wrl
+      (at (xyz 0 0 0))
+      (scale (xyz 1 1 1))
+      (rotate (xyz 0 0 0))
+    )
+  )
   (module Connector_PinSocket_2.54mm:PinSocket_1x08_P2.54mm_Vertical (layer F.Cu)
     (at 24.13 110.49 180)
@@
   )
   (module Capacitor_SMD:C_0603_1608Metric (layer F.Cu)
-    (at 81.28 110.49)
+    (at 67.31 99.06 180)
     (descr "Capacitor SMD 0603 (1608 Metric), square (rectangular) end terminal, IPC_7351 nominal, (Body size source: IPC-SM-782 page 76, https://www.pcb-3d.com/wordpress/wp-content/uploads/ipc-sm-782a_amendment_1_and_2.pdf), generated with kicad-footprint-generator")
     (tags capacitor)
@@
       (effects (font (size 0.4 0.4) (thickness 0.06)))
     )
-    (pad 1 smd roundrect (at -0.775 0) (size 0.9 0.95) (layers F.Cu F.Paste F.Mask) (roundrect_rratio 0.25)
+    (pad 1 smd roundrect (at -0.775 0 180) (size 0.9 0.95) (layers F.Cu F.Paste F.Mask) (roundrect_rratio 0.25)
       (net 5 +3V3))
-    (pad 2 smd roundrect (at 0.775 0) (size 0.9 0.95) (layers F.Cu F.Paste F.Mask) (roundrect_rratio 0.25)
+    (pad 2 smd roundrect (at 0.775 0 180) (size 0.9 0.95) (layers F.Cu F.Paste F.Mask) (roundrect_rratio 0.25)
       (net 4 GND))
     (model ${KISYS3DMOD}/Capacitor_SMD.3dshapes/C_0603_1608Metric.wrl
@@
   )
   (module Capacitor_SMD:C_0805_2012Metric (layer F.Cu)
-    (at 67.31 102.87 180)
+    (at 67.31 106.68 180)
     (descr "Capacitor SMD 0805 (2012 Metric), square (rectangular) end terminal, IPC_7351 nominal, (Body size source: IPC-SM-782 page 76, https://www.pcb-3d.com/wordpress/wp-content/uploads/ipc-sm-782a_amendment_1_and_2.pdf, https://docs.google.com/spreadsheets/d/1BsfQQcO9C6DZCsRaXUlFlo91Tg2WpOkGARC1WS5S8t0/edit?usp=sharing), generated with kicad-footprint-generator")
     (tags capacitor)
@@
   )
   (module Capacitor_SMD:C_0603_1608Metric (layer F.Cu)
-    (at 66.815 99.06 180)
+    (at 66.815 102.87 180)
     (descr "Capacitor SMD 0603 (1608 Metric), square (rectangular) end terminal, IPC_7351 nominal, (Body size source: IPC-SM-782 page 76, https://www.pcb-3d.com/wordpress/wp-content/uploads/ipc-sm-782a_amendment_1_and_2.pdf), generated with kicad-footprint-generator")
     (tags capacitor)
@@
   )
   (module Package_TO_SOT_SMD:SOT-23 (layer F.Cu)
-    (at 87.63 96.52)
+    (at 77.2 100.01 180)
     (descr "SOT-23, Standard")
     (tags SOT-23)
@@
       (effects (font (size 0.5 0.5) (thickness 0.075)))
     )
-    (pad 3 smd rect (at 1 0) (size 0.9 0.8) (layers F.Cu F.Paste F.Mask)
+    (pad 3 smd rect (at 1 0 180) (size 0.9 0.8) (layers F.Cu F.Paste F.Mask)
       (net 35 "Net-(Q1-Pad3)"))
-    (pad 2 smd rect (at -1 0.95) (size 0.9 0.8) (layers F.Cu F.Paste F.Mask)
-      (net 4 GND))
-    (pad 1 smd rect (at -1 -0.95) (size 0.9 0.8) (layers F.Cu F.Paste F.Mask)
+    (pad 2 smd rect (at -1 0.95 180) (size 0.9 0.8) (layers F.Cu F.Paste F.Mask)
+      (net 4 GND))
+    (pad 1 smd rect (at -1 -0.95 180) (size 0.9 0.8) (layers F.Cu F.Paste F.Mask)
       (net 36 "Net-(Q1-Pad1)"))
     (model ${KISYS3DMOD}/Package_TO_SOT_SMD.3dshapes/SOT-23.wrl
@@
   )
   (module Resistor_SMD:R_0805_2012Metric (layer F.Cu)
-    (at 81.6375 114.3)
+    (at 72.0325 106.68)
     (descr "Resistor SMD 0805 (2012 Metric), square (rectangular) end terminal, IPC_7351 nominal, (Body size source: IPC-SM-782 page 72, https://www.pcb-3d.com/wordpress/wp-content/uploads/ipc-sm-782a_amendment_1_and_2.pdf), generated with kicad-footprint-generator")
     (tags resistor)
@@
   )
   (module Resistor_SMD:R_0805_2012Metric (layer F.Cu)
-    (at 87.63 114.3 180)
+    (at 72.39 102.87 180)
     (descr "Resistor SMD 0805 (2012 Metric), square (rectangular) end terminal, IPC_7351 nominal, (Body size source: IPC-SM-782 page 72, https://www.pcb-3d.com/wordpress/wp-content/uploads/ipc-sm-782a_amendment_1_and_2.pdf), generated with kicad-footprint-generator")
     (tags resistor)
@@
   )
   (module 147873-1:SW_147873-1 (layer F.Cu)
-    (at 85.23 87.63)
+    (at 73.52 87.63)
     (fp_text reference SWBOOTesp1 (at -2.321135 -2.562461) (layer F.SilkS)
       (effects (font (size 0.630773 0.630773) (thickness 0.015)))

Commit message: wires
Parts:
- J3: footprint Connector_PinHeader_1.00mm:PinHeader_1x03_P1.00mm_Vertical -> Connector_PinSocket_2.54mm:PinSocket_1x03_P2.54mm_Vertical
- moved J3 51.1 mm to (55.9, 87.6), turned to 90 degrees
- moved C5 34.9 mm to (96.0, 83.8)
- moved R1 34.9 mm to (101.2, 87.6)
- moved R2 34.9 mm to (108.0, 87.6)
- moved C1 34.9 mm to (96.2, 76.2)
- moved R6 34.9 mm to (108.0, 90.6)
- moved C2 34.9 mm to (96.5, 80.0)
- moved C3 34.9 mm to (96.5, 87.6)
- moved C4 34.9 mm to (95.6, 72.4)
- moved R4 34.9 mm to (101.6, 83.8)
- moved Q2 33.1 mm to (107.6, 75.2), turned to 90 degrees
- moved Q1 31.1 mm to (101.3, 80.3), turned to 90 degrees
- moved Blue1 29.2 mm to (121.9, 87.6)
- moved Cout1 29.2 mm to (138.4, 121.9)
- moved Cout2 29.2 mm to (114.6, 121.9)
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Routing:
- net GND: track 0.00 -> 31.5 mm

Commit message: wires
Parts:
- moved R7 48.1 mm to (65.7, 95.2)
- moved Q2 47.9 mm to (66.0, 99.1)
- moved R6 42.3 mm to (65.7, 91.4)
- moved C3 37.7 mm to (64.8, 108.0), turned to 0 degrees
- moved R1 37.7 mm to (69.5, 108.0)
- moved J2 1.27 mm to (69.8, 116.8)
- moved J4 1.27 mm to (58.4, 116.8)
- moved R10 1.27 mm to (67.3, 113.0)
- moved R11 1.27 mm to (63.5, 113.0)
Routing:
- net GND: track 31.5 -> 0.00 mm

Commit message: wires
Parts:
- moved R2 46.2 mm to (64.8, 104.1)
- moved R3 44.4 mm to (76.2, 87.6), turned to 180 degrees
- moved C4 43.7 mm to (73.7, 110.2), turned to 270 degrees
- moved Q1 35.5 mm to (71.1, 99.1), turned to 0 degrees
- moved C2 28.3 mm to (70.6, 91.4)
- moved C5 27.9 mm to (70.6, 95.2)
- moved C1 27.9 mm to (70.8, 87.6)
- moved R4 26.9 mm to (76.2, 92.7), turned to 0 degrees
- moved ENesp1 23.9 mm to (78.7, 109.2), turned to 90 degrees
- moved SWBOOTesp1 11.4 mm to (78.7, 99.1), turned to 90 degrees
Changed lines of the file:
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@@
   )
   (module Resistor_SMD:R_0805_2012Metric (layer F.Cu)
-    (at 107.95 87.63)
+    (at 64.77 104.14)
     (descr "Resistor SMD 0805 (2012 Metric), square (rectangular) end terminal, IPC_7351 nominal, (Body size source: IPC-SM-782 page 72, https://www.pcb-3d.com/wordpress/wp-content/uploads/ipc-sm-782a_amendment_1_and_2.pdf), generated with kicad-footprint-generator")
     (tags resistor)
@@
   )
   (module Capacitor_SMD:C_0805_2012Metric (layer F.Cu)
-    (at 96.2 76.2 180)
+    (at 70.8 87.63 180)
     (descr "Capacitor SMD 0805 (2012 Metric), square (rectangular) end terminal, IPC_7351 nominal, (Body size source: IPC-SM-782 page 76, https://www.pcb-3d.com/wordpress/wp-content/uploads/ipc-sm-782a_amendment_1_and_2.pdf, https://docs.google.com/spreadsheets/d/1BsfQQcO9C6DZCsRaXUlFlo91Tg2WpOkGARC1WS5S8t0/edit?usp=sharing), generated with kicad-footprint-generator")
     (tags capacitor)
@@
   )
   (module Capacitor_SMD:C_0603_1608Metric (layer F.Cu)
-    (at 96.52 80.01 180)
+    (at 70.625 91.44 180)
     (descr "Capacitor SMD 0603 (1608 Metric), square (rectangular) end terminal, IPC_7351 nominal, (Body size source: IPC-SM-782 page 76, https://www.pcb-3d.com/wordpress/wp-content/uploads/ipc-sm-782a_amendment_1_and_2.pdf), generated with kicad-footprint-generator")
     (tags capacitor)
@@
   )
   (module Capacitor_SMD:C_0805_2012Metric (layer F.Cu)
-    (at 95.57 72.39 180)
+    (at 73.66 110.17 270)
     (descr "Capacitor SMD 0805 (2012 Metric), square (rectangular) end terminal, IPC_7351 nominal, (Body size source: IPC-SM-782 page 76, https://www.pcb-3d.com/wordpress/wp-content/uploads/ipc-sm-782a_amendment_1_and_2.pdf, https://docs.google.com/spreadsheets/d/1BsfQQcO9C6DZCsRaXUlFlo91Tg2WpOkGARC1WS5S8t0/edit?usp=sharing), generated with kicad-footprint-generator")
     (tags capacitor)
     (attr smd)
-    (fp_text reference C4 (at 0 -1.68) (layer F.SilkS)
-      (effects (font (size 1 1) (thickness 0.15)))
-    )
-    (fp_text value 0.1uF (at 0 1.68) (layer F.Fab)
+    (fp_text reference C4 (at 0 -1.68 90) (layer F.SilkS)
+      (effects (font (size 1 1) (thickness 0.15)))
+    )
+    (fp_text value 0.1uF (at 0 1.68 90) (layer F.Fab)
       (effects (font (size 1 1) (thickness 0.15)))
     )
@@
     (fp_line (start 1.7 -0.98) (end 1.7 0.98) (layer F.CrtYd) (width 0.05))
     (fp_line (start 1.7 0.98) (end -1.7 0.98) (layer F.CrtYd) (width 0.05))
-    (fp_text user %R (at 0 0) (layer F.Fab)
-      (effects (font (size 0.5 0.5) (thickness 0.08)))
-    )
-    (pad 1 smd roundrect (at -0.95 0 180) (size 1 1.45) (layers F.Cu F.Paste F.Mask) (roundrect_rratio 0.25)
+    (fp_text user %R (at 0 0 90) (layer F.Fab)
+      (effects (font (size 0.5 0.5) (thickness 0.08)))
+    )
+    (pad 1 smd roundrect (at -0.95 0 270) (size 1 1.45) (layers F.Cu F.Paste F.Mask) (roundrect_rratio 0.25)
       (net 7 "Net-(C4-Pad1)"))
-    (pad 2 smd roundrect (at 0.95 0 180) (size 1 1.45) (layers F.Cu F.Paste F.Mask) (roundrect_rratio 0.25)
+    (pad 2 smd roundrect (at 0.95 0 270) (size 1 1.45) (layers F.Cu F.Paste F.Mask) (roundrect_rratio 0.25)
       (net 4 GND))
     (model ${KISYS3DMOD}/Capacitor_SMD.3dshapes/C_0805_2012Metric.wrl
@@
   )
   (module Capacitor_SMD:C_0603_1608Metric (layer F.Cu)
-    (at 96.025 83.82 180)
+    (at 70.625 95.25 180)
     (descr "Capacitor SMD 0603 (1608 Metric), square (rectangular) end terminal, IPC_7351 nominal, (Body size source: IPC-SM-782 page 76, https://www.pcb-3d.com/wordpress/wp-content/uploads/ipc-sm-782a_amendment_1_and_2.pdf), generated with kicad-footprint-generator")
     (tags capacitor)
@@
   )
   (module 147873-1:SW_147873-1 (layer F.Cu)
-    (at 68.44 87.63)
-    (fp_text reference ENesp1 (at -2.321135 -2.562461) (layer F.SilkS)
+    (at 78.74 109.22 90)
+    (fp_text reference ENesp1 (at -2.321135 -2.562461 90) (layer F.SilkS)
       (effects (font (size 0.630773 0.630773) (thickness 0.015)))
     )
-    (fp_text value 147873-1 (at 0.082076 2.52334) (layer F.Fab)
+    (fp_text value 147873-1 (at 0.082076 2.52334 90) (layer F.Fab)
       (effects (font (size 0.630505 0.630505) (thickness 0.015)))
     )
@@
     (fp_line (start -3 1.75) (end 3 1.75) (layer F.Fab) (width 0.127))
     (fp_line (start -3 -1.75) (end -3 1.75) (layer F.Fab) (width 0.127))
-    (pad 2 smd rect (at 2.4 0) (size 2.8 2.2) (layers F.Cu F.Paste F.Mask)
+    (pad 2 smd rect (at 2.4 0 90) (size 2.8 2.2) (layers F.Cu F.Paste F.Mask)
       (net 7 "Net-(C4-Pad1)"))
-    (pad 1 smd rect (at -2.4 0) (size 2.8 2.2) (layers F.Cu F.Paste F.Mask)
+    (pad 1 smd rect (at -2.4 0 90) (size 2.8 2.2) (layers F.Cu F.Paste F.Mask)
       (net 4 GND))
   )
@@
   )
   (module Package_TO_SOT_SMD:SOT-23 (layer F.Cu)
-    (at 101.28 80.28 90)
+    (at 71.12 99.06)
     (descr "SOT-23, Standard")
     (tags SOT-23)
     (attr smd)
-    (fp_text reference Q1 (at 0 -2.5 90) (layer F.SilkS)
-      (effects (font (size 1 1) (thickness 0.15)))
-    )
-    (fp_text value BSS138 (at 0 2.5 90) (layer F.Fab)
+    (fp_text reference Q1 (at 0 -2.5) (layer F.SilkS)
+      (effects (font (size 1 1) (thickness 0.15)))
+    )
+    (fp_text value BSS138 (at 0 2.5) (layer F.Fab)
       (effects (font (size 1 1) (thickness 0.15)))
     )
@@
     (fp_line (start -0.15 -1.52) (end 0.7 -1.52) (layer F.Fab) (width 0.1))
     (fp_line (start -0.7 -0.95) (end -0.7 1.5) (layer F.Fab) (width 0.1))
-    (fp_text user %R (at 0 0) (layer F.Fab)
+    (fp_text user %R (at 0 0 90) (layer F.Fab)
       (effects (font (size 0.5 0.5) (thickness 0.075)))
     )
-    (pad 3 smd rect (at 1 0 90) (size 0.9 0.8) (layers F.Cu F.Paste F.Mask)
+    (pad 3 smd rect (at 1 0) (size 0.9 0.8) (layers F.Cu F.Paste F.Mask)
       (net 35 "Net-(Q1-Pad3)"))
-    (pad 2 smd rect (at -1 0.95 90) (size 0.9 0.8) (layers F.Cu F.Paste F.Mask)
-      (net 4 GND))
-    (pad 1 smd rect (at -1 -0.95 90) (size 0.9 0.8) (layers F.Cu F.Paste F.Mask)
+    (pad 2 smd rect (at -1 0.95) (size 0.9 0.8) (layers F.Cu F.Paste F.Mask)
+      (net 4 GND))
+    (pad 1 smd rect (at -1 -0.95) (size 0.9 0.8) (layers F.Cu F.Paste F.Mask)
       (net 36 "Net-(Q1-Pad1)"))
     (model ${KISYS3DMOD}/Package_TO_SOT_SMD.3dshapes/SOT-23.wrl
@@
   )
   (module Resistor_SMD:R_0805_2012Metric (layer F.Cu)
-    (at 116.84 105.41)
+    (at 76.2 87.63 180)
     (descr "Resistor SMD 0805 (2012 Metric), square (rectangular) end terminal, IPC_7351 nominal, (Body size source: IPC-SM-782 page 72, https://www.pcb-3d.com/wordpress/wp-content/uploads/ipc-sm-782a_amendment_1_and_2.pdf), generated with kicad-footprint-generator")
     (tags resistor)
@@
       (effects (font (size 0.5 0.5) (thickness 0.08)))
     )
-    (pad 2 smd roundrect (at 0.9125 0) (size 1.025 1.4) (layers F.Cu F.Paste F.Mask) (roundrect_rratio 0.243902)
-      (net 4 GND))
-    (pad 1 smd roundrect (at -0.9125 0) (size 1.025 1.4) (layers F.Cu F.Paste F.Mask) (roundrect_rratio 0.243902)
+    (pad 2 smd roundrect (at 0.9125 0 180) (size 1.025 1.4) (layers F.Cu F.Paste F.Mask) (roundrect_rratio 0.243902)
+      (net 4 GND))
+    (pad 1 smd roundrect (at -0.9125 0 180) (size 1.025 1.4) (layers F.Cu F.Paste F.Mask) (roundrect_rratio 0.243902)
       (net 8 "Net-(C5-Pad1)"))
     (model ${KISYS3DMOD}/Resistor_SMD.3dshapes/R_0805_2012Metric.wrl
@@
   )
   (module Resistor_SMD:R_0805_2012Metric (layer F.Cu)
-    (at 101.6 83.82 180)
+    (at 76.2 92.71)
     (descr "Resistor SMD 0805 (2012 Metric), square (rectangular) end terminal, IPC_7351 nominal, (Body size source: IPC-SM-782 page 72, https://www.pcb-3d.com/wordpress/wp-content/uploads/ipc-sm-782a_amendment_1_and_2.pdf), generated with kicad-footprint-generator")
     (tags resistor)
@@
       (effects (font (size 0.5 0.5) (thickness 0.08)))
     )
-    (pad 1 smd roundrect (at -0.9125 0 180) (size 1.025 1.4) (layers F.Cu F.Paste F.Mask) (roundrect_rratio 0.243902)
+    (pad 1 smd roundrect (at -0.9125 0) (size 1.025 1.4) (layers F.Cu F.Paste F.Mask) (roundrect_rratio 0.243902)
       (net 36 "Net-(Q1-Pad1)"))
-    (pad 2 smd roundrect (at 0.9125 0 180) (size 1.025 1.4) (layers F.Cu F.Paste F.Mask) (roundrect_rratio 0.243902)
+    (pad 2 smd roundrect (at 0.9125 0) (size 1.025 1.4) (layers F.Cu F.Paste F.Mask) (roundrect_rratio 0.243902)
       (net 8 "Net-(C5-Pad1)"))
     (model ${KISYS3DMOD}/Resistor_SMD.3dshapes/R_0805_2012Metric.wrl
@@
   )
   (module 147873-1:SW_147873-1 (layer F.Cu)
-    (at 78.6 87.63)
-    (fp_text reference SWBOOTesp1 (at -2.321135 -2.562461) (layer F.SilkS)
+    (at 78.74 99.06 90)
+    (fp_text reference SWBOOTesp1 (at -2.321135 -2.562461 90) (layer F.SilkS)
       (effects (font (size 0.630773 0.630773) (thickness 0.015)))
     )
-    (fp_text value 147873-1 (at 0.082076 2.52334) (layer F.Fab)
+    (fp_text value 147873-1 (at 0.082076 2.52334 90) (layer F.Fab)
       (effects (font (size 0.630505 0.630505) (thickness 0.015)))
     )
@@
     (fp_line (start 4.05 2) (end 4.05 -2) (layer F.CrtYd) (width 0.05))
     (fp_line (start 4.05 -2) (end -4.05 -2) (layer F.CrtYd) (width 0.05))
-    (pad 1 smd rect (at -2.4 0) (size 2.8 2.2) (layers F.Cu F.Paste F.Mask)
+    (pad 1 smd rect (at -2.4 0 90) (size 2.8 2.2) (layers F.Cu F.Paste F.Mask)
       (net 5 +3V3))
-    (pad 2 smd rect (at 2.4 0) (size 2.8 2.2) (layers F.Cu F.Paste F.Mask)
+    (pad 2 smd rect (at 2.4 0 90) (size 2.8 2.2) (layers F.Cu F.Paste F.Mask)
       (net 8 "Net-(C5-Pad1)"))
   )

Commit message: wires
Parts:
- moved J1 95.6 mm to (118.1, 92.7), turned to 0 degrees
- moved R9 66.5 mm to (73.7, 116.8), turned to 90 degrees
- moved C6 60.0 mm to (81.0, 90.2), turned to 0 degrees
- moved Blue1 52.1 mm to (78.7, 116.8), turned to 180 degrees
- moved R8 51.1 mm to (83.8, 116.8), turned to 270 degrees
- moved LedRed1 49.0 mm to (90.2, 116.8), turned to 0 degrees
- moved R5 46.2 mm to (71.1, 104.1), turned to 0 degrees
- moved Cout1 41.5 mm to (100.3, 105.4)
- moved U1 40.4 mm to (88.9, 105.4)
- moved BZ1 34.9 mm to (88.9, 92.7)
- moved U2 28.0 mm to (106.0, 92.5)
- moved Cin1 27.0 mm to (109.8, 102.9)
- moved Cin2 26.9 mm to (109.8, 111.8)
- moved Cout2 15.3 mm to (100.6, 115.6), turned to 180 degrees
