File: pruebakicad/prueba.kicad_pcb (KiCad board)
At the start: 2 copper layers, 36 parts, among them J1 Conn_01x08_RC522, J2 Conn_01x04_MountingPin, J3 Conn_01x03, J4 Conn_2Rows-15Pins, J5 Conn_01x04, Q1 BSS138, Q2 BSS138, U1 TLV1117-33, U2 TLV1117-50, U3 ESP32-WROOM-32

Commit message: pistas
Parts:
- added J6: Conn_01x02, Connector_PinSocket_2.54mm:PinSocket_1x02_P2.54mm_Vertical, F.Cu at (109.2, 118.1)
Routing:
- net /RST: track 0.00 -> 80.7 mm, vias 0 -> 1
- net /MOSI: track 0.00 -> 79.6 mm, vias 0 -> 1
- net /SDAspi: track 0.00 -> 72.4 mm, vias 0 -> 1
- net /MISO: track 0.00 -> 72.2 mm, vias 0 -> 1
- net /SCK: track 0.00 -> 67.8 mm, vias 0 -> 1
- net /BUZ: track 0.00 -> 32.9 mm, vias 0 -> 1
- net Net-(C5-Pad1): track 0.00 -> 31.0 mm
- net /esp32-wroom/EN: track 0.00 -> 29.2 mm
- net /IO13: track 0.00 -> 27.9 mm
- net Net-(LedRed1-Pad2): track 0.00 -> 19.4 mm
- net Net-(C4-Pad1): track 0.00 -> 16.2 mm
- net Net-(Q1-Pad3): track 0.00 -> 11.4 mm
- net /IO32: track 0.00 -> 8.16 mm
- net /IO25: track 0.00 -> 8.16 mm
- net /sensVP: track 0.00 -> 8.16 mm
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
Commit message: ruteo completo
Parts:
- moved R11 3.92 mm to (67.3, 113.9), turned to 90 degrees
- moved R10 3.81 mm to (63.5, 113.0), turned to 270 degrees
- moved J2 2.54 mm to (69.8, 119.4)
- moved J3 2.54 mm to (55.9, 85.1)
- moved J4 2.54 mm to (58.4, 119.4)
- moved J5 2.54 mm to (43.2, 85.1)
Connections:
- U1 pad 4: (no net) -> +3V3
- U2 pad 2: +5V -> Net-(U2-Pad2)
- U2 pad 4: (no net) -> +5V
Routing:
- net +5V: track 0.00 -> 186.5 mm
- net +3V3: track 8.16 -> 187.3 mm, vias 0 -> 2
- net GND: track 7.63 -> 79.3 mm, vias 0 -> 7
- net +12V: track 0.00 -> 40.2 mm
- net /SCLi2c: track 4.71 -> 23.6 mm
- net /SDAi2c: track 4.19 -> 13.5 mm
- net /RST: track 80.7 -> 88.6 mm
- net /MISO: track 72.2 -> 76.8 mm
- net /MOSI: track 79.6 -> 84.0 mm
- net /SCK: track 67.8 -> 72.1 mm
- net /sensVN: track 5.09 -> 7.63 mm
- net /IO35: track 5.09 -> 7.63 mm
- net /IO33: track 5.09 -> 7.63 mm
- net /IO27: track 5.62 -> 8.16 mm
- net /IO26: track 5.09 -> 7.63 mm
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- added copper zone on F.Cu, net GND

Commit message: gnd
Routing:
- net GND: track 79.3 -> 48.8 mm, vias 7 -> 0
- net +3V3: track 187.3 -> 188.5 mm
- net Net-(C4-Pad1): track 16.2 -> 17.2 mm
- net Net-(Q2-Pad1): track 8.27 -> 7.30 mm
- net /SDAi2c: track 13.5 -> 14.4 mm
- net /IO13: track 28.7 -> 28.0 mm

Commit message: asss
Connections:
- J6 pad 1: +12V -> Net-(J6-Pad1)
- J6 pad 2: GND -> Net-(J6-Pad2)
Routing:
- net /SCK: track 72.1 -> 68.3 mm
- net /MOSI: track 84.0 -> 80.7 mm
- net /MISO: track 76.8 -> 73.8 mm
- net /RST: track 88.6 -> 86.0 mm
- net +3V3: track 188.5 -> 186.4 mm
- net /BUZ: track 34.8 -> 33.2 mm
- net +5V: track 186.5 -> 187.9 mm

Commit message: asdsad
Parts:
- J6: footprint Connector_PinSocket_2.54mm:PinSocket_1x02_P2.54mm_Vertical -> Connector_BarrelJack:BarrelJack_CUI_PJ-063AH_Horizontal
- moved J6 6.68 mm to (110.2, 111.5), turned to 0 degrees
- moved Cin2 5.08 mm to (109.7, 106.7)
- moved Cin1 2.79 mm to (109.8, 100.1)
- moved Cout2 2.55 mm to (98.0, 115.6)
- moved R8 0.72 mm to (84.3, 116.3), turned to 180 degrees
Connections:
- J6 pad 1: Net-(J6-Pad1) -> +12V
- J6 pad 2: Net-(J6-Pad2) -> GND
Routing:
- net GND: track 48.8 -> 0.40 mm
- net +3V3: track 186.4 -> 172.7 mm
- net +12V: track 40.2 -> 34.1 mm
- net Net-(Blue1-Pad1): track 4.52 -> 3.95 mm
- net /IO13: track 28.0 -> 27.5 mm

Commit message: tierras
Parts:
- J2, J5: footprint Connector_PinSocket_2.54mm:PinSocket_1x04_P2.54mm_Vertical -> Connector_PinSocket_2.54mm:PinSocket_1x04_P2.54mm_Horizontal
- J3: footprint Connector_PinSocket_2.54mm:PinSocket_1x03_P2.54mm_Vertical -> Connector_PinSocket_2.54mm:PinSocket_1x03_P2.54mm_Horizontal
- J4: footprint Connector_PinSocket_2.54mm:PinSocket_2x07_P2.54mm_Vertical -> Connector_PinSocket_2.54mm:PinSocket_2x07_P2.54mm_Horizontal
- moved J4 17.0 mm to (42.7, 113.0), turned to 90 degrees
- moved LedRed1 13.2 mm to (77.0, 117.0), turned to 270 degrees
- moved J2 8.98 mm to (61.7, 115.6), turned to 90 degrees
- moved J5 8.76 mm to (50.8, 89.4), turned to 270 degrees
- moved Cout2 6.36 mm to (91.7, 115.3)
- moved Blue1 6.35 mm to (85.1, 117.0), turned to 90 degrees
- moved J6 6.35 mm to (104.0, 112.8)
- moved J3 5.76 mm to (59.7, 89.4), turned to 270 degrees
- moved R8 3.61 mm to (80.8, 117.0), turned to 270 degrees
- moved R11 2.80 mm to (66.5, 111.3)
- moved C4 2.73 mm to (73.7, 107.4)
- moved R10 1.78 mm to (63.5, 111.3)
- moved C2 1.28 mm to (69.3, 91.4)
- moved C6 0.07 mm to (81.0, 90.2), turned to 180 degrees
Connections:
- C6 pad 1: +3V3 -> GND
- C6 pad 2: GND -> +3V3
- J2 pad 1: +5V -> GND
- J2 pad 2: /SDAi2c -> +5V
- J2 pad 3: /SCLi2c -> /SDAi2c
- J2 pad 4: GND -> /SCLi2c
- J3 pad 1: /OBS -> GND
- J3 pad 2: GND -> +5V
- J3 pad 3: +5V -> /OBS
- J4 pad 1: +5V -> GND
- J4 pad 10: /sensVN -> /IO32
- J4 pad 11: +3V3 -> /IO26
- J4 pad 12: +3V3 -> /IO25
- J4 pad 13: GND -> +5V
- J4 pad 14: GND -> /IO27
- J4 pad 2: /IO27 -> GND
- J4 pad 3: /IO25 -> +3V3
- J4 pad 4: /IO26 -> +3V3
- J4 pad 5: /IO32 -> /sensVN
- J4 pad 6: /IO33 -> /sensVP
- J4 pad 7: /IO34 -> /IO35
- J4 pad 8: /IO35 -> /IO34
- J4 pad 9: /sensVP -> /IO33
- J5 pad 1: +3V3 -> GND
- J5 pad 2: /TXD0 -> /RXD0
- J5 pad 3: /RXD0 -> /TXD0
- J5 pad 4: GND -> +3V3
Routing:
- net Net-(LedRed1-Pad2): track 19.4 -> 3.72 mm
- net +3V3: track 172.7 -> 164.3 mm
- net +5V: track 188.1 -> 194.7 mm, vias 0 -> 1
- net /IO13: track 27.5 -> 33.6 mm
- net /OBS: track 8.40 -> 3.55 mm
- net Net-(Q1-Pad3): track 11.4 -> 15.8 mm
- net /TXD0: track 7.65 -> 3.33 mm
- net /RXD0: track 7.87 -> 3.55 mm
- net /sensVP: track 10.7 -> 6.68 mm
- net /IO34: track 10.7 -> 6.68 mm
- net /IO33: track 7.63 -> 3.61 mm
- net /IO26: track 7.63 -> 3.61 mm
- net /IO32: track 10.7 -> 6.68 mm
- net /IO25: track 10.7 -> 6.68 mm
- net /sensVN: track 7.63 -> 3.61 mm
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- added copper zone on B.Cu, net GND
Other:
- board outline added: 94.1 x 42.4 mm
