File: pruebakicad/esp.sch (KiCad schematic (older format))
At the start: 19 parts, among them U1 ESP32-WROOM-32

Commit message: footprints
Footprints added
Parts:
- Blue1: footprint (none) -> LED_SMD:LED_0805_2012Metric
- C1, C3, C4: footprint (none) -> Capacitor_SMD:C_0805_2012Metric
- C2, C5: footprint (none) -> Capacitor_SMD:C_0603_1608Metric
- R1, R3, R4, R5, R6, R7, R8: footprint (none) -> Resistor_SMD:R_0805_2012Metric
- gave numbers to parts that had none: 2
- renumbered BOOTesp to BOOTesp1, ENesp to ENesp1, U1 to U3
Connections:
- wire segments 82 -> 81
Changed lines of the file:
@@
 	6550 2400 6800 2400
 $Comp
-L RF_Module:ESP32-WROOM-32 U1
+L RF_Module:ESP32-WROOM-32 U3
 U 1 1 60779D57
 P 5950 2800
-F 0 "U1" H 5950 4381 50  0000 C CNN
+F 0 "U3" H 5950 4381 50  0000 C CNN
 F 1 "ESP32-WROOM-32" H 5950 4290 50  0000 C CNN
 F 2 "RF_Module:ESP32-WROOM-32" H 5950 1300 50  0001 C CNN
@@
 F 0 "Blue1" H 3000 1693 50  0000 C CNN
 F 1 "LED_Small" H 3000 1784 50  0000 C CNN
-F 2 "" V 3000 1900 50  0001 C CNN
+F 2 "LED_SMD:LED_0805_2012Metric" V 3000 1900 50  0001 C CNN
 F 3 "~" V 3000 1900 50  0001 C CNN
 	1    3000 1900
@@
 F 0 "R8" H 3182 1954 50  0000 R CNN
 F 1 "220" H 3182 2045 50  0000 R CNN
-F 2 "" H 3250 2000 50  0001 C CNN
+F 2 "Resistor_SMD:R_0805_2012Metric" H 3250 2000 50  0001 C CNN
 F 3 "~" H 3250 2000 50  0001 C CNN
 	1    3250 2000
@@
 P 3250 2150
 AR Path="/607F1C44" Ref="#PWR?"  Part="1"
-AR Path="/6077B277/607F1C44" Ref="#PWR?"  Part="1"
-F 0 "#PWR?" H 3250 1900 50  0001 C CNN
+AR Path="/6077B277/607F1C44" Ref="#PWR0115"  Part="1"
+F 0 "#PWR0115" H 3250 1900 50  0001 C CNN
 F 1 "GND" H 3255 1977 50  0000 C CNN
 F 2 "" H 3250 2150 50  0001 C CNN
@@
 	2900 1900 2750 1900
 $Comp
-L power:+3V3 #PWR?
+L power:+3V3 #PWR0116
 U 1 1 607F479D
 P 900 1100
-F 0 "#PWR?" H 900 950 50  0001 C CNN
+F 0 "#PWR0116" H 900 950 50  0001 C CNN
 F 1 "+3V3" H 915 1273 50  0000 C CNN
 F 2 "" H 900 1100 50  0001 C CNN
@@
 F 0 "C1" H 1242 1346 50  0000 L CNN
 F 1 "0.1uF" H 1242 1255 50  0000 L CNN
-F 2 "" H 1150 1300 50  0001 C CNN
+F 2 "Capacitor_SMD:C_0805_2012Metric" H 1150 1300 50  0001 C CNN
 F 3 "~" H 1150 1300 50  0001 C CNN
 	1    1150 1300
@@
 F 0 "C2" H 1742 1346 50  0000 L CNN
 F 1 "10uF" H 1742 1255 50  0000 L CNN
-F 2 "" H 1650 1300 50  0001 C CNN
+F 2 "Capacitor_SMD:C_0603_1608Metric" H 1650 1300 50  0001 C CNN
 F 3 "~" H 1650 1300 50  0001 C CNN
 	1    1650 1300
@@
 	5950 1400 5950 1150
 $Comp
-L power:+3.3V #PWR?
+L power:+3.3V #PWR0117
 U 1 1 607F93CE
 P 5950 1150
-F 0 "#PWR?" H 5950 1000 50  0001 C CNN
+F 0 "#PWR0117" H 5950 1000 50  0001 C CNN
 F 1 "+3.3V" H 5965 1323 50  0000 C CNN
 F 2 "" H 5950 1150 50  0001 C CNN
@@
 F 0 "C3" H 1492 2746 50  0000 L CNN
 F 1 "1uF" H 1492 2655 50  0000 L CNN
-F 2 "" H 1400 2700 50  0001 C CNN
+F 2 "Capacitor_SMD:C_0805_2012Metric" H 1400 2700 50  0001 C CNN
 F 3 "~" H 1400 2700 50  0001 C CNN
 	1    1400 2700
@@
 $EndComp
 $Comp
-L power:GND #PWR?
+L power:GND #PWR0118
 U 1 1 607FA4E3
 P 1400 2850
-F 0 "#PWR?" H 1400 2600 50  0001 C CNN
+F 0 "#PWR0118" H 1400 2600 50  0001 C CNN
 F 1 "GND" H 1405 2677 50  0000 C CNN
 F 2 "" H 1400 2850 50  0001 C CNN
@@
 $EndComp
 $Comp
-L power:GND #PWR?
+L power:GND #PWR0119
 U 1 1 607F5DBA
 P 1400 1550
-F 0 "#PWR?" H 1400 1300 50  0001 C CNN
+F 0 "#PWR0119" H 1400 1300 50  0001 C CNN
 F 1 "GND" H 1405 1377 50  0000 C CNN
 F 2 "" H 1400 1550 50  0001 C CNN
@@
 F 0 "R1" H 1332 2304 50  0000 R CNN
 F 1 "10k" H 1332 2395 50  0000 R CNN
-F 2 "" H 1400 2350 50  0001 C CNN
+F 2 "Resistor_SMD:R_0805_2012Metric" H 1400 2350 50  0001 C CNN
 F 3 "~" H 1400 2350 50  0001 C CNN
 	1    1400 2350
@@
 $EndComp
 $Comp
-L power:+3.3V #PWR?
+L power:+3.3V #PWR0120
 U 1 1 607FBCCF
 P 1400 2150
-F 0 "#PWR?" H 1400 2000 50  0001 C CNN
+F 0 "#PWR0120" H 1400 2000 50  0001 C CNN
 F 1 "+3.3V" H 1415 2323 50  0000 C CNN
 F 2 "" H 1400 2150 50  0001 C CNN
@@
 	1200 4150 1250 4150
 $Comp
-L power:GND #PWR?
+L power:GND #PWR0121
 U 1 1 60806CDE
 P 1200 4550
-F 0 "#PWR?" H 1200 4300 50  0001 C CNN
+F 0 "#PWR0121" H 1200 4300 50  0001 C CNN
 F 1 "GND" H 1205 4377 50  0000 C CNN
 F 2 "" H 1200 4550 50  0001 C CNN
@@
 	2000 4150 1900 4150
 $Comp
-L Switch:SW_DIP_x01 ENesp
+L Switch:SW_DIP_x01 ENesp1
 U 1 1 60802839
 P 1550 4150
-F 0 "ENesp" H 1550 4417 50  0000 C CNN
+F 0 "ENesp1" H 1550 4417 50  0000 C CNN
 F 1 "SW_DIP_x01" H 1550 4326 50  0000 C CNN
 F 2 "" H 1550 4150 50  0001 C CNN
@@
 EN
 $Comp
-L Switch:SW_DIP_x01 BOOTesp
+L Switch:SW_DIP_x01 BOOTesp1
 U 1 1 60811B80
 P 1250 5250
-F 0 "BOOTesp" H 1250 5517 50  0000 C CNN
+F 0 "BOOTesp1" H 1250 5517 50  0000 C CNN
 F 1 "SW_DIP_x01" H 1250 5426 50  0000 C CNN
 F 2 "" H 1250 5250 50  0001 C CNN
@@
 $EndComp
 $Comp
-L power:+3.3V #PWR?
+L power:+3.3V #PWR0123
 U 1 1 607F7FA8
 P 1850 1050
-F 0 "#PWR?" H 1850 900 50  0001 C CNN
+F 0 "#PWR0123" H 1850 900 50  0001 C CNN
 F 1 "+3.3V" H 1865 1223 50  0000 C CNN
 F 2 "" H 1850 1050 50  0001 C CNN
@@
 F 0 "R5" V 2154 5850 50  0000 C CNN
 F 1 "1k" V 2245 5850 50  0000 C CNN
-F 2 "" H 2350 5850 50  0001 C CNN
+F 2 "Resistor_SMD:R_0805_2012Metric" H 2350 5850 50  0001 C CNN
 F 3 "~" H 2350 5850 50  0001 C CNN
 	1    2350 5850
@@
 F 0 "C4" H 1642 4496 50  0000 L CNN
 F 1 "0.1uF" H 1642 4405 50  0000 L CNN
-F 2 "" H 1550 4450 50  0001 C CNN
+F 2 "Capacitor_SMD:C_0805_2012Metric" H 1550 4450 50  0001 C CNN
 F 3 "~" H 1550 4450 50  0001 C CNN
 	1    1550 4450
@@
 F 0 "C5" H 1892 5546 50  0000 L CNN
 F 1 "1nF" H 1892 5455 50  0000 L CNN
-F 2 "" H 1800 5500 50  0001 C CNN
+F 2 "Capacitor_SMD:C_0603_1608Metric" H 1800 5500 50  0001 C CNN
 F 3 "~" H 1800 5500 50  0001 C CNN
 	1    1800 5500
@@
 	0    1    1    0
 $EndComp
-Wire Wire Line
-	1900 4450 2100 4450
-Connection ~ 1900 4450
-$Comp
-L power:+3.3V #PWR?
+$Comp
+L power:+3.3V #PWR0124
 U 1 1 60820D78
 P 800 5100
-F 0 "#PWR?" H 800 4950 50  0001 C CNN
+F 0 "#PWR0124" H 800 4950 50  0001 C CNN
 F 1 "+3.3V" H 815 5273 50  0000 C CNN
 F 2 "" H 800 5100 50  0001 C CNN
@@
 F 0 "R3" V 1454 5500 50  0000 C CNN
 F 1 "10k" V 1545 5500 50  0000 C CNN
-F 2 "" H 1650 5500 50  0001 C CNN
+F 2 "Resistor_SMD:R_0805_2012Metric" H 1650 5500 50  0001 C CNN
 F 3 "~" H 1650 5500 50  0001 C CNN
 	1    1650 5500
@@
 F 0 "R4" V 2104 4800 50  0000 C CNN
 F 1 "1k" V 2195 4800 50  0000 C CNN
-F 2 "" H 2300 4800 50  0001 C CNN
+F 2 "Resistor_SMD:R_0805_2012Metric" H 2300 4800 50  0001 C CNN
 F 3 "~" H 2300 4800 50  0001 C CNN
 	1    2300 4800
@@
 	1800 5250 2100 5250
 $Comp
-L Transistor_FET:BSS138 Q?
+L Transistor_FET:BSS138 Q1
 U 1 1 6083E5A9
 P 2700 4800
-F 0 "Q?" H 2904 4846 50  0000 L CNN
+F 0 "Q1" H 2904 4846 50  0000 L CNN
 F 1 "BSS138" H 2904 4755 50  0000 L CNN
 F 2 "Package_TO_SOT_SMD:SOT-23" H 2900 4725 50  0001 L CIN
@@
 $EndComp
 $Comp
-L Transistor_FET:BSS138 Q?
+L Transistor_FET:BSS138 Q2
 U 1 1 60842FF2
 P 2750 5850
-F 0 "Q?" H 2954 5896 50  0000 L CNN
+F 0 "Q2" H 2954 5896 50  0000 L CNN
 F 1 "BSS138" H 2954 5805 50  0000 L CNN
 F 2 "Package_TO_SOT_SMD:SOT-23" H 2950 5775 50  0001 L CIN
@@
 	2500 4800 2400 4800
 $Comp
-L power:GND #PWR?
+L power:GND #PWR0125
 U 1 1 60851FCE
 P 2800 5100
-F 0 "#PWR?" H 2800 4850 50  0001 C CNN
+F 0 "#PWR0125" H 2800 4850 50  0001 C CNN
 F 1 "GND" H 2805 4927 50  0000 C CNN
 F 2 "" H 2800 5100 50  0001 C CNN
@@
 	2800 5100 2800 5000
 $Comp
-L power:GND #PWR?
+L power:GND #PWR0126
 U 1 1 60853F50
 P 2850 6150
-F 0 "#PWR?" H 2850 5900 50  0001 C CNN
+F 0 "#PWR0126" H 2850 5900 50  0001 C CNN
 F 1 "GND" H 2855 5977 50  0000 C CNN
 F 2 "" H 2850 6150 50  0001 C CNN
@@
 F 0 "R6" V 2854 4550 50  0000 C CNN
 F 1 "1k" V 2945 4550 50  0000 C CNN
-F 2 "" H 3050 4550 50  0001 C CNN
+F 2 "Resistor_SMD:R_0805_2012Metric" H 3050 4550 50  0001 C CNN
 F 3 "~" H 3050 4550 50  0001 C CNN
 	1    3050 4550
@@
 F 0 "R7" V 2904 5600 50  0000 C CNN
 F 1 "1k" V 2995 5600 50  0000 C CNN
-F 2 "" H 3100 5600 50  0001 C CNN
+F 2 "Resistor_SMD:R_0805_2012Metric" H 3100 5600 50  0001 C CNN
 F 3 "~" H 3100 5600 50  0001 C CNN
 	1    3100 5600
@@
 	2100 4800 2100 5250
 $Comp
-L power:GND #PWR?
+L power:GND #PWR0127
 U 1 1 60876589
 P 1700 5750
-F 0 "#PWR?" H 1700 5500 50  0001 C CNN
+F 0 "#PWR0127" H 1700 5500 50  0001 C CNN
 F 1 "GND" H 1705 5577 50  0000 C CNN
 F 2 "" H 1700 5750 50  0001 C CNN

Commit message: footprints
Finished footprints
Parts:
- removed BOOTesp1, ENesp1: SW_DIP_x01, symbol Switch:SW_DIP_x01
- added ENesp1, SWBOOTesp1: 147873-1, 147873-1:SW_147873-1, symbol Elementos:147873-1
- R6, R7: value 1k -> 0R; footprint Resistor_SMD:R_0805_2012Metric -> (none)
Connections:
- net +3V3: now also SWBOOTesp1.1
- net GND: now also ENesp1.1
- net at C4.1, R2.2: now also ENesp1.2
- net at C5.1, R3.1, R4.2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: now also SWBOOTesp1.2
Changed lines of the file:
@@
 Text Label 1450 2550 0    50   ~ 0
 EN
-Wire Wire Line
-	1200 4150 1250 4150
 $Comp
 L power:GND #PWR0121
@@
 Wire Wire Line
 	2000 4150 1900 4150
-$Comp
-L Switch:SW_DIP_x01 ENesp1
-U 1 1 60802839
-P 1550 4150
-F 0 "ENesp1" H 1550 4417 50  0000 C CNN
-F 1 "SW_DIP_x01" H 1550 4326 50  0000 C CNN
-F 2 "" H 1550 4150 50  0001 C CNN
-F 3 "~" H 1550 4150 50  0001 C CNN
-	1    1550 4150
-	1    0    0    -1
-$EndComp
 Wire Wire Line
 	2200 4150 2450 4150
 Text Label 2300 4150 0    50   ~ 0
 EN
-$Comp
-L Switch:SW_DIP_x01 BOOTesp1
-U 1 1 60811B80
-P 1250 5250
-F 0 "BOOTesp1" H 1250 5517 50  0000 C CNN
-F 1 "SW_DIP_x01" H 1250 5426 50  0000 C CNN
-F 2 "" H 1250 5250 50  0001 C CNN
-F 3 "~" H 1250 5250 50  0001 C CNN
-	1    1250 5250
-	1    0    0    -1
-$EndComp
 $Comp
 L power:+3.3V #PWR0123
@@
 	1900 4450 1900 4150
 Connection ~ 1900 4150
-Wire Wire Line
-	1900 4150 1850 4150
 Wire Notes Line
 	600  600  600  3200
@@
 $EndComp
 Wire Wire Line
-	950  5250 800  5250
-Wire Wire Line
 	800  5250 800  5100
-Wire Wire Line
-	1550 5250 1650 5250
 $Comp
 L Device:R_Small R3
@@
 P 3050 4550
 F 0 "R6" V 2854 4550 50  0000 C CNN
-F 1 "1k" V 2945 4550 50  0000 C CNN
-F 2 "Resistor_SMD:R_0805_2012Metric" H 3050 4550 50  0001 C CNN
+F 1 "0R" V 2945 4550 50  0000 C CNN
+F 2 "" H 3050 4550 50  0001 C CNN
 F 3 "~" H 3050 4550 50  0001 C CNN
 	1    3050 4550
@@
 P 3100 5600
 F 0 "R7" V 2904 5600 50  0000 C CNN
-F 1 "1k" V 2995 5600 50  0000 C CNN
-F 2 "Resistor_SMD:R_0805_2012Metric" H 3100 5600 50  0001 C CNN
+F 1 "0R" V 2995 5600 50  0000 C CNN
+F 2 "" H 3100 5600 50  0001 C CNN
 F 3 "~" H 3100 5600 50  0001 C CNN
 	1    3100 5600
@@
 Text HLabel 6800 1900 2    50   Input ~ 0
 RXD0
+$Comp
+L Elementos:147873-1 ENesp1
+U 1 1 608A77D8
+P 1550 4150
+F 0 "ENesp1" H 1550 4352 50  0000 C CNN
+F 1 "147873-1" H 1550 4261 50  0000 C CNN
+F 2 "147873-1:SW_147873-1" H 1550 4150 50  0001 L BNN
+F 3 "" H 1550 4150 50  0001 L BNN
+F 4 "147873-1" H 1550 4150 50  0001 L BNN "Comment"
+	1    1550 4150
+	1    0    0    -1
+$EndComp
+$Comp
+L Elementos:147873-1 SWBOOTesp1
+U 1 1 608A8447
+P 1250 5250
+F 0 "SWBOOTesp1" H 1250 5452 50  0000 C CNN
+F 1 "147873-1" H 1250 5361 50  0000 C CNN
+F 2 "147873-1:SW_147873-1" H 1250 5250 50  0001 L BNN
+F 3 "" H 1250 5250 50  0001 L BNN
+F 4 "147873-1" H 1250 5250 50  0001 L BNN "Comment"
+	1    1250 5250
+	1    0    0    -1
+$EndComp
+Wire Wire Line
+	1200 4150 1350 4150
+Wire Wire Line
+	1750 4150 1900 4150
+Wire Wire Line
+	800  5250 1050 5250
+Wire Wire Line
+	1450 5250 1650 5250
 $EndSCHEMATC

Commit message: wires
Parts:
- R2, R6, R7: footprint (none) -> Resistor_SMD:R_0805_2012Metric
Changed lines of the file:
@@
 F 0 "R2" V 1904 4150 50  0000 C CNN
 F 1 "0R" V 1995 4150 50  0000 C CNN
-F 2 "" H 2100 4150 50  0001 C CNN
+F 2 "Resistor_SMD:R_0805_2012Metric" H 2100 4150 50  0001 C CNN
 F 3 "~" H 2100 4150 50  0001 C CNN
 	1    2100 4150
@@
 F 0 "R6" V 2854 4550 50  0000 C CNN
 F 1 "0R" V 2945 4550 50  0000 C CNN
-F 2 "" H 3050 4550 50  0001 C CNN
+F 2 "Resistor_SMD:R_0805_2012Metric" H 3050 4550 50  0001 C CNN
 F 3 "~" H 3050 4550 50  0001 C CNN
 	1    3050 4550
@@
 F 0 "R7" V 2904 5600 50  0000 C CNN
 F 1 "0R" V 2995 5600 50  0000 C CNN
-F 2 "" H 3100 5600 50  0001 C CNN
+F 2 "Resistor_SMD:R_0805_2012Metric" H 3100 5600 50  0001 C CNN
 F 3 "~" H 3100 5600 50  0001 C CNN
 	1    3100 5600
