File: pruebakicad/esp.sch (KiCad schematic (older format))
At the start: 19 parts, among them Q1 BSS138, Q2 BSS138, U3 ESP32-WROOM-32

Commit message: holes
Parts:
- Led2: renamed from Blue1; value LED_Small -> LED_BLUE
Changed lines of the file:
@@
 P 3000 1900
 AR Path="/607F1C37" Ref="Blue?"  Part="1"
-AR Path="/6077B277/607F1C37" Ref="Blue1"  Part="1"
-F 0 "Blue1" H 3000 1693 50  0000 C CNN
-F 1 "LED_Small" H 3000 1784 50  0000 C CNN
+AR Path="/6077B277/607F1C37" Ref="Led2"  Part="1"
+F 0 "Led2" H 3000 1693 50  0000 C CNN
+F 1 "LED_BLUE" H 3000 1784 50  0000 C CNN
 F 2 "LED_SMD:LED_0805_2012Metric" V 3000 1900 50  0001 C CNN
 F 3 "~" V 3000 1900 50  0001 C CNN

Commit message: Gerber
Parts:
- renumbered SWBOOTesp1 to BOOT1, ENesp1 to EN1
Changed lines of the file:
@@
 RXD0
 $Comp
-L Elementos:147873-1 ENesp1
+L Elementos:147873-1 EN1
 U 1 1 608A77D8
 P 1550 4150
-F 0 "ENesp1" H 1550 4352 50  0000 C CNN
+F 0 "EN1" H 1550 4352 50  0000 C CNN
 F 1 "147873-1" H 1550 4261 50  0000 C CNN
 F 2 "147873-1:SW_147873-1" H 1550 4150 50  0001 L BNN
@@
 $EndComp
 $Comp
-L Elementos:147873-1 SWBOOTesp1
+L Elementos:147873-1 BOOT1
 U 1 1 608A8447
 P 1250 5250
-F 0 "SWBOOTesp1" H 1250 5452 50  0000 C CNN
+F 0 "BOOT1" H 1250 5452 50  0000 C CNN
 F 1 "147873-1" H 1250 5361 50  0000 C CNN
 F 2 "147873-1:SW_147873-1" H 1250 5250 50  0001 L BNN
