File: pruebakicad/out.sch (KiCad schematic (older format))
At the start: 9 parts, among them J1 Conn_01x08_RC522, J2 Conn_01x04_MountingPin, J3 Conn_01x03, J4 Conn_2Rows-15Pins, J5 Conn_01x04

Commit message: wires
Parts:
- J1: footprint Connector_PinHeader_1.00mm:PinHeader_1x08_P1.00mm_Vertical -> Connector_PinSocket_2.54mm:PinSocket_1x08_P2.54mm_Vertical
- J2, J5: footprint Connector_PinHeader_1.00mm:PinHeader_1x04_P1.00mm_Vertical -> Connector_PinSocket_2.54mm:PinSocket_1x04_P2.54mm_Vertical
- J4: footprint Connector_PinSocket_2.54mm:PinSocket_2x09_P2.54mm_Vertical -> Connector_PinSocket_2.54mm:PinSocket_2x07_P2.54mm_Vertical
Changed lines of the file:
@@
 F 0 "J2" H 4838 4514 50  0000 L CNN
 F 1 "Conn_01x04_MountingPin" H 4838 4423 50  0000 L CNN
-F 2 "Connector_PinHeader_1.00mm:PinHeader_1x04_P1.00mm_Vertical" H 4750 4600 50  0001 C CNN
+F 2 "Connector_PinSocket_2.54mm:PinSocket_1x04_P2.54mm_Vertical" H 4750 4600 50  0001 C CNN
 F 3 "~" H 4750 4600 50  0001 C CNN
 	1    4750 4600
@@
 F 0 "J1" H 4750 3800 50  0000 C CNN
 F 1 "Conn_01x08_RC522" H 4750 3700 50  0000 C CNN
-F 2 "Connector_PinHeader_1.00mm:PinHeader_1x08_P1.00mm_Vertical" H 4750 3300 50  0001 C CNN
+F 2 "Connector_PinSocket_2.54mm:PinSocket_1x08_P2.54mm_Vertical" H 4750 3300 50  0001 C CNN
 F 3 "~" H 4750 3300 50  0001 C CNN
 	1    4750 3300
@@
 F 0 "J4" H 6850 3967 50  0000 C CNN
 F 1 "Conn_2Rows-15Pins" H 6850 3876 50  0000 C CNN
-F 2 "Connector_PinSocket_2.54mm:PinSocket_2x09_P2.54mm_Vertical" H 6800 3350 50  0001 C CNN
+F 2 "Connector_PinSocket_2.54mm:PinSocket_2x07_P2.54mm_Vertical" H 6800 3350 50  0001 C CNN
 F 3 "~" H 6800 3350 50  0001 C CNN
 	1    6800 3350
@@
 F 0 "J5" H 7480 4742 50  0000 L CNN
 F 1 "Conn_01x04" H 7480 4651 50  0000 L CNN
-F 2 "Connector_PinHeader_1.00mm:PinHeader_1x04_P1.00mm_Vertical" H 7400 4750 50  0001 C CNN
+F 2 "Connector_PinSocket_2.54mm:PinSocket_1x04_P2.54mm_Vertical" H 7400 4750 50  0001 C CNN
 F 3 "~" H 7400 4750 50  0001 C CNN
 	1    7400 4750

Commit message: wires
Parts:
- J3: footprint Connector_PinHeader_1.00mm:PinHeader_1x03_P1.00mm_Vertical -> Connector_PinSocket_2.54mm:PinSocket_1x03_P2.54mm_Vertical
Changed lines of the file:
@@
 F 0 "J3" H 4830 5642 50  0000 L CNN
 F 1 "Conn_01x03" H 4830 5551 50  0000 L CNN
-F 2 "Connector_PinHeader_1.00mm:PinHeader_1x03_P1.00mm_Vertical" H 4750 5600 50  0001 C CNN
+F 2 "Connector_PinSocket_2.54mm:PinSocket_1x03_P2.54mm_Vertical" H 4750 5600 50  0001 C CNN
 F 3 "~" H 4750 5600 50  0001 C CNN
 	1    4750 5600

Commit message: wires
Changed lines of the file:
@@
 	1    0    0    -1
 $EndComp
-Text HLabel 5900 2800 0    50   Input ~ 0
-IO13
-Text HLabel 5900 2900 0    50   Input ~ 0
-IO15
-Text HLabel 5900 3100 0    50   Input ~ 0
-IO16
-Text HLabel 5900 3000 0    50   Input ~ 0
-IO17
 Text HLabel 7300 3050 2    50   Input ~ 0
 IO26

Commit message: tierras
Parts:
- J2, J5: footprint Connector_PinSocket_2.54mm:PinSocket_1x04_P2.54mm_Vertical -> Connector_PinSocket_2.54mm:PinSocket_1x04_P2.54mm_Horizontal
- J3: footprint Connector_PinSocket_2.54mm:PinSocket_1x03_P2.54mm_Vertical -> Connector_PinSocket_2.54mm:PinSocket_1x03_P2.54mm_Horizontal
- J4: footprint Connector_PinSocket_2.54mm:PinSocket_2x07_P2.54mm_Vertical -> Connector_PinSocket_2.54mm:PinSocket_2x07_P2.54mm_Horizontal
Connections:
- net +3V3: now also C6.2, J4.3 (IO13), J4.4 (IO32), J5.4 (GND); no longer C6.1, J4.11 (IO25), J4.12 (sensVP), J5.1 (VCC)
- net +5V: now also J2.2 (SDAi2c), J3.2 (GND), J4.13 (IO26); no longer J2.1 (VCC), J3.3 (VCC), J4.1 (3.3V)
- net GND: now also C6.1, J2.1 (VCC), J3.1 (OBS), J4.1 (3.3V), J4.2 (IO27), J5.1 (VCC); no longer C6.2, J2.4 (GND), J3.2 (GND), J4.13 (IO26), J4.14 (sensVN), J5.4 (GND)
- net IO25: now also J4.12 (sensVP); no longer J4.3 (IO13)
- net IO26: now also J4.11 (IO25); no longer J4.4 (IO32)
- net IO27: now also J4.14 (sensVN); no longer J4.2 (IO27)
- net IO32: now also J4.10 (IO35); no longer J4.5 (IO15)
- net IO33: now also J4.9 (IO17); no longer J4.6 (IO33)
- net IO34: now also J4.8 (IO34); no longer J4.7 (IO16)
- net IO35: now also J4.7 (IO16); no longer J4.8 (IO34)
- net OBS: now also J3.3 (VCC); no longer J3.1 (OBS)
- net RXD0: now also J5.2 (TXD0); no longer J5.3 (RXD0)
- net SCLi2c: now also J2.4 (GND); no longer J2.3 (SCLi2c)
- net SDAi2c: now also J2.3 (SCLi2c); no longer J2.2 (SDAi2c)
- net TXD0: now also J5.3 (RXD0); no longer J5.2 (TXD0)
- net sensVN: now also J4.5 (IO15); no longer J4.10 (IO35)
- net sensVP: now also J4.6 (IO33); no longer J4.9 (IO17)
Other:
- moved on the sheet: J2, J4, R10, R11
