File: pruebakicad/Reguladores.sch (KiCad schematic (older format))
At the start: 8 parts

Commit message: footprints
Footprints added
Parts:
- Cin1, Cin2: footprint (none) -> Capacitor_SMD:CP_Elec_4x5.7
- Cout1, Cout2: footprint (none) -> Capacitor_SMD:CP_Elec_6.3x5.9
- LedRed1: renamed from LedRed; footprint (none) -> LED_SMD:LED_0805_2012Metric
- R9: value 2k -> 220; footprint (none) -> Resistor_SMD:R_0805_2012Metric
- U1, U2: renamed from U?; footprint (none) -> Package_TO_SOT_SMD:SOT-223
Changed lines of the file:
@@
 P 4600 2000
 AR Path="/6088E1E3" Ref="U?"  Part="1"
-AR Path="/608889A3/6088E1E3" Ref="U?"  Part="1"
-F 0 "U?" H 4600 2242 50  0000 C CNN
+AR Path="/608889A3/6088E1E3" Ref="U1"  Part="1"
+F 0 "U1" H 4600 2242 50  0000 C CNN
 F 1 "TLV1117-33" H 4600 2151 50  0000 C CNN
-F 2 "" H 4600 2000 50  0001 C CNN
+F 2 "Package_TO_SOT_SMD:SOT-223" H 4600 2000 50  0001 C CNN
 F 3 "http://www.ti.com/lit/ds/symlink/tlv1117.pdf" H 4600 2000 50  0001 C CNN
 	1    4600 2000
@@
 P 4650 4250
 AR Path="/6088E1E9" Ref="U?"  Part="1"
-AR Path="/608889A3/6088E1E9" Ref="U?"  Part="1"
-F 0 "U?" H 4650 4492 50  0000 C CNN
+AR Path="/608889A3/6088E1E9" Ref="U2"  Part="1"
+F 0 "U2" H 4650 4492 50  0000 C CNN
 F 1 "TLV1117-50" H 4650 4401 50  0000 C CNN
-F 2 "" H 4650 4250 50  0001 C CNN
+F 2 "Package_TO_SOT_SMD:SOT-223" H 4650 4250 50  0001 C CNN
 F 3 "http://www.ti.com/lit/ds/symlink/tlv1117.pdf" H 4650 4250 50  0001 C CNN
 	1    4650 4250
@@
 P 4000 1950
 AR Path="/6088E1EF" Ref="#PWR?"  Part="1"
-AR Path="/608889A3/6088E1EF" Ref="#PWR?"  Part="1"
-F 0 "#PWR?" H 4000 1800 50  0001 C CNN
+AR Path="/608889A3/6088E1EF" Ref="#PWR0128"  Part="1"
+F 0 "#PWR0128" H 4000 1800 50  0001 C CNN
 F 1 "+12V" H 4015 2123 50  0000 C CNN
 F 2 "" H 4000 1950 50  0001 C CNN
@@
 P 3950 4150
 AR Path="/6088E1F5" Ref="#PWR?"  Part="1"
-AR Path="/608889A3/6088E1F5" Ref="#PWR?"  Part="1"
-F 0 "#PWR?" H 3950 4000 50  0001 C CNN
+AR Path="/608889A3/6088E1F5" Ref="#PWR0129"  Part="1"
+F 0 "#PWR0129" H 3950 4000 50  0001 C CNN
 F 1 "+12V" H 3965 4323 50  0000 C CNN
 F 2 "" H 3950 4150 50  0001 C CNN
@@
 P 4650 4700
 AR Path="/6088E1FD" Ref="#PWR?"  Part="1"
-AR Path="/608889A3/6088E1FD" Ref="#PWR?"  Part="1"
-F 0 "#PWR?" H 4650 4450 50  0001 C CNN
+AR Path="/608889A3/6088E1FD" Ref="#PWR0130"  Part="1"
+F 0 "#PWR0130" H 4650 4450 50  0001 C CNN
 F 1 "GND" H 4655 4527 50  0000 C CNN
 F 2 "" H 4650 4700 50  0001 C CNN
@@
 P 4600 2450
 AR Path="/6088E203" Ref="#PWR?"  Part="1"
-AR Path="/608889A3/6088E203" Ref="#PWR?"  Part="1"
-F 0 "#PWR?" H 4600 2200 50  0001 C CNN
+AR Path="/608889A3/6088E203" Ref="#PWR0131"  Part="1"
+F 0 "#PWR0131" H 4600 2200 50  0001 C CNN
 F 1 "GND" H 4605 2277 50  0000 C CNN
 F 2 "" H 4600 2450 50  0001 C CNN
@@
 F 0 "Cin1" H 4115 2346 50  0000 L CNN
 F 1 "10u" H 4115 2255 50  0000 L CNN
-F 2 "" H 4000 2300 50  0001 C CNN
+F 2 "Capacitor_SMD:CP_Elec_4x5.7" H 4000 2300 50  0001 C CNN
 F 3 "~" H 4000 2300 50  0001 C CNN
 	1    4000 2300
@@
 F 0 "Cout1" H 5315 2296 50  0000 L CNN
 F 1 "100u" H 5315 2205 50  0000 L CNN
-F 2 "" H 5200 2250 50  0001 C CNN
+F 2 "Capacitor_SMD:CP_Elec_6.3x5.9" H 5200 2250 50  0001 C CNN
 F 3 "~" H 5200 2250 50  0001 C CNN
 	1    5200 2250
@@
 P 4000 2550
 AR Path="/6088E21C" Ref="#PWR?"  Part="1"
-AR Path="/608889A3/6088E21C" Ref="#PWR?"  Part="1"
-F 0 "#PWR?" H 4000 2300 50  0001 C CNN
+AR Path="/608889A3/6088E21C" Ref="#PWR0132"  Part="1"
+F 0 "#PWR0132" H 4000 2300 50  0001 C CNN
 F 1 "GND" H 4005 2377 50  0000 C CNN
 F 2 "" H 4000 2550 50  0001 C CNN
@@
 P 5200 2500
 AR Path="/6088E222" Ref="#PWR?"  Part="1"
-AR Path="/608889A3/6088E222" Ref="#PWR?"  Part="1"
-F 0 "#PWR?" H 5200 2250 50  0001 C CNN
+AR Path="/608889A3/6088E222" Ref="#PWR0133"  Part="1"
+F 0 "#PWR0133" H 5200 2250 50  0001 C CNN
 F 1 "GND" H 5205 2327 50  0000 C CNN
 F 2 "" H 5200 2500 50  0001 C CNN
@@
 P 3950 4700
 AR Path="/6088E228" Ref="#PWR?"  Part="1"
-AR Path="/608889A3/6088E228" Ref="#PWR?"  Part="1"
-F 0 "#PWR?" H 3950 4450 50  0001 C CNN
+AR Path="/608889A3/6088E228" Ref="#PWR0134"  Part="1"
+F 0 "#PWR0134" H 3950 4450 50  0001 C CNN
 F 1 "GND" H 3955 4527 50  0000 C CNN
 F 2 "" H 3950 4700 50  0001 C CNN
@@
 P 5200 4750
 AR Path="/6088E22E" Ref="#PWR?"  Part="1"
-AR Path="/608889A3/6088E22E" Ref="#PWR?"  Part="1"
-F 0 "#PWR?" H 5200 4500 50  0001 C CNN
+AR Path="/608889A3/6088E22E" Ref="#PWR0135"  Part="1"
+F 0 "#PWR0135" H 5200 4500 50  0001 C CNN
 F 1 "GND" H 5205 4577 50  0000 C CNN
 F 2 "" H 5200 4750 50  0001 C CNN
@@
 F 0 "Cin2" H 4065 4546 50  0000 L CNN
 F 1 "10u" H 4065 4455 50  0000 L CNN
-F 2 "" H 3950 4500 50  0001 C CNN
+F 2 "Capacitor_SMD:CP_Elec_4x5.7" H 3950 4500 50  0001 C CNN
 F 3 "~" H 3950 4500 50  0001 C CNN
 	1    3950 4500
@@
 F 0 "Cout2" H 5315 4546 50  0000 L CNN
 F 1 "100u" H 5315 4455 50  0000 L CNN
-F 2 "" H 5200 4500 50  0001 C CNN
+F 2 "Capacitor_SMD:CP_Elec_6.3x5.9" H 5200 4500 50  0001 C CNN
 F 3 "~" H 5200 4500 50  0001 C CNN
 	1    5200 4500
@@
 P 5200 1900
 AR Path="/6088E248" Ref="#PWR?"  Part="1"
-AR Path="/608889A3/6088E248" Ref="#PWR?"  Part="1"
-F 0 "#PWR?" H 5200 1750 50  0001 C CNN
+AR Path="/608889A3/6088E248" Ref="#PWR0136"  Part="1"
+F 0 "#PWR0136" H 5200 1750 50  0001 C CNN
 F 1 "+3V3" H 5215 2073 50  0000 C CNN
 F 2 "" H 5200 1900 50  0001 C CNN
@@
 P 5200 4150
 AR Path="/6088E24E" Ref="#PWR?"  Part="1"
-AR Path="/608889A3/6088E24E" Ref="#PWR?"  Part="1"
-F 0 "#PWR?" H 5200 4000 50  0001 C CNN
+AR Path="/608889A3/6088E24E" Ref="#PWR0137"  Part="1"
+F 0 "#PWR0137" H 5200 4000 50  0001 C CNN
 F 1 "+5V" H 5215 4323 50  0000 C CNN
 F 2 "" H 5200 4150 50  0001 C CNN
@@
 	5200 4350 5200 4250
 $Comp
-L Device:LED_Small LedRed
+L Device:LED_Small LedRed1
 U 1 1 6089055D
 P 5750 4850
-F 0 "LedRed" V 5796 4780 50  0000 R CNN
+F 0 "LedRed1" V 5796 4780 50  0000 R CNN
 F 1 "LED_Small" V 5705 4780 50  0000 R CNN
-F 2 "" V 5750 4850 50  0001 C CNN
+F 2 "LED_SMD:LED_0805_2012Metric" V 5750 4850 50  0001 C CNN
 F 3 "~" V 5750 4850 50  0001 C CNN
 	1    5750 4850
@@
 	5750 4250 5750 4400
 $Comp
-L power:GND #PWR?
+L power:GND #PWR0138
 U 1 1 60891458
 P 5750 5050
-F 0 "#PWR?" H 5750 4800 50  0001 C CNN
+F 0 "#PWR0138" H 5750 4800 50  0001 C CNN
 F 1 "GND" H 5755 4877 50  0000 C CNN
 F 2 "" H 5750 5050 50  0001 C CNN
@@
 AR Path="/608889A3/60893024" Ref="R9"  Part="1"
 F 0 "R9" V 5554 4500 50  0000 C CNN
-F 1 "2k" V 5645 4500 50  0000 C CNN
-F 2 "" H 5750 4500 50  0001 C CNN
+F 1 "220" V 5645 4500 50  0000 C CNN
+F 2 "Resistor_SMD:R_0805_2012Metric" H 5750 4500 50  0001 C CNN
 F 3 "~" H 5750 4500 50  0001 C CNN
 	1    5750 4500

Commit message: pistas
Parts:
- added J?: Conn_01x02, Connector_PinSocket_2.54mm:PinSocket_1x02_P2.54mm_Vertical, symbol Connector_Generic:Conn_01x02
Connections:
- net +12V: now also J?.1 (Pin_1)
- net GND: now also J?.2 (Pin_2)
Changed lines of the file:
@@
 Wire Wire Line
 	5750 4600 5750 4750
+$Comp
+L Connector_Generic:Conn_01x02 J?
+U 1 1 60E48AF7
+P 3350 3200
+F 0 "J?" H 3430 3192 50  0000 L CNN
+F 1 "Conn_01x02" H 3430 3101 50  0000 L CNN
+F 2 "Connector_PinSocket_2.54mm:PinSocket_1x02_P2.54mm_Vertical" H 3350 3200 50  0001 C CNN
+F 3 "~" H 3350 3200 50  0001 C CNN
+	1    3350 3200
+	1    0    0    -1
+$EndComp
+Wire Wire Line
+	3150 3200 2900 3200
+Wire Wire Line
+	3150 3300 2900 3300
+$Comp
+L power:+12V #PWR?
+U 1 1 60E4A1A7
+P 2900 3200
+AR Path="/60E4A1A7" Ref="#PWR?"  Part="1"
+AR Path="/608889A3/60E4A1A7" Ref="#PWR?"  Part="1"
+F 0 "#PWR?" H 2900 3050 50  0001 C CNN
+F 1 "+12V" H 2915 3373 50  0000 C CNN
+F 2 "" H 2900 3200 50  0001 C CNN
+F 3 "" H 2900 3200 50  0001 C CNN
+	1    2900 3200
+	1    0    0    -1
+$EndComp
+$Comp
+L power:GND #PWR?
+U 1 1 60E4A59F
+P 2900 3300
+AR Path="/60E4A59F" Ref="#PWR?"  Part="1"
+AR Path="/608889A3/60E4A59F" Ref="#PWR?"  Part="1"
+F 0 "#PWR?" H 2900 3050 50  0001 C CNN
+F 1 "GND" H 2905 3127 50  0000 C CNN
+F 2 "" H 2900 3300 50  0001 C CNN
+F 3 "" H 2900 3300 50  0001 C CNN
+	1    2900 3300
+	1    0    0    -1
+$EndComp
 $EndSCHEMATC

Commit message: ruteo completo
Parts:
- U1: symbol Regulator_Linear:TLV1117-33 -> Elementos:LM1117-3.3
- U2: symbol Regulator_Linear:TLV1117-50 -> Elementos:TLV1117-50
- gave numbers to parts that had none: 1
Connections:
- net +3V3: now also U1.4 (VO)
- net +5V: now also U2.4 (VO); no longer U2.2 (VO)
- no-connect marks 0 -> 1
Changed lines of the file:
@@
 $Descr A4 11693 8268
 encoding utf-8
-Sheet 4 4
+Sheet 3 4
 Title ""
 Date ""
@@
 $EndDescr
 $Comp
-L Regulator_Linear:TLV1117-33 U?
+L Elementos:LM1117-3.3 U?
 U 1 1 6088E1E3
 P 4600 2000
@@
 $EndComp
 $Comp
-L Regulator_Linear:TLV1117-50 U?
+L Elementos:TLV1117-50 U?
 U 1 1 6088E1E9
 P 4650 4250
@@
 $EndComp
 Wire Wire Line
-	4900 2000 5200 2000
-Wire Wire Line
 	5200 2000 5200 2100
 Wire Wire Line
@@
 $EndComp
 Wire Wire Line
-	5200 4250 4950 4250
+	5200 4250 5050 4250
 Wire Wire Line
 	3950 4250 4350 4250
@@
 	5750 4600 5750 4750
 $Comp
-L Connector_Generic:Conn_01x02 J?
+L Connector_Generic:Conn_01x02 J6
 U 1 1 60E48AF7
 P 3350 3200
-F 0 "J?" H 3430 3192 50  0000 L CNN
+F 0 "J6" H 3430 3192 50  0000 L CNN
 F 1 "Conn_01x02" H 3430 3101 50  0000 L CNN
 F 2 "Connector_PinSocket_2.54mm:PinSocket_1x02_P2.54mm_Vertical" H 3350 3200 50  0001 C CNN
@@
 P 2900 3200
 AR Path="/60E4A1A7" Ref="#PWR?"  Part="1"
-AR Path="/608889A3/60E4A1A7" Ref="#PWR?"  Part="1"
-F 0 "#PWR?" H 2900 3050 50  0001 C CNN
+AR Path="/608889A3/60E4A1A7" Ref="#PWR0140"  Part="1"
+F 0 "#PWR0140" H 2900 3050 50  0001 C CNN
 F 1 "+12V" H 2915 3373 50  0000 C CNN
 F 2 "" H 2900 3200 50  0001 C CNN
@@
 P 2900 3300
 AR Path="/60E4A59F" Ref="#PWR?"  Part="1"
-AR Path="/608889A3/60E4A59F" Ref="#PWR?"  Part="1"
-F 0 "#PWR?" H 2900 3050 50  0001 C CNN
+AR Path="/608889A3/60E4A59F" Ref="#PWR0142"  Part="1"
+F 0 "#PWR0142" H 2900 3050 50  0001 C CNN
 F 1 "GND" H 2905 3127 50  0000 C CNN
 F 2 "" H 2900 3300 50  0001 C CNN
@@
 	1    0    0    -1
 $EndComp
+Wire Wire Line
+	4950 4400 5050 4400
+Wire Wire Line
+	5050 4400 5050 4250
+Wire Wire Line
+	5000 2150 5000 2000
+Wire Wire Line
+	4900 2150 5000 2150
+Wire Wire Line
+	5000 2000 5200 2000
+Wire Wire Line
+	4900 2000 5000 2000
+Connection ~ 5000 2000
+NoConn ~ 4950 4250
 $EndSCHEMATC

Commit message: asss
Parts:
- J6: symbol Connector_Generic:Conn_01x02 -> Connector:Barrel_Jack
Changed lines of the file:
@@
 	5750 4600 5750 4750
 $Comp
-L Connector_Generic:Conn_01x02 J6
+L Connector:Barrel_Jack J6
 U 1 1 60E48AF7
 P 3350 3200

Commit message: asdsad
Parts:
- J6: footprint Connector_PinSocket_2.54mm:PinSocket_1x02_P2.54mm_Vertical -> Connector_BarrelJack:BarrelJack_CUI_PJ-063AH_Horizontal
Other:
- moved on the sheet: J6
Changed lines of the file:
@@
 L Connector:Barrel_Jack J6
 U 1 1 60E48AF7
-P 3350 3200
-F 0 "J6" H 3430 3192 50  0000 L CNN
-F 1 "Conn_01x02" H 3430 3101 50  0000 L CNN
-F 2 "Connector_PinSocket_2.54mm:PinSocket_1x02_P2.54mm_Vertical" H 3350 3200 50  0001 C CNN
-F 3 "~" H 3350 3200 50  0001 C CNN
-	1    3350 3200
-	1    0    0    -1
+P 3650 3200
+F 0 "J6" H 3600 3500 50  0000 L CNN
+F 1 "Conn_01x02" H 3450 3450 50  0000 L CNN
+F 2 "Connector_BarrelJack:BarrelJack_CUI_PJ-063AH_Horizontal" H 3650 3200 50  0001 C CNN
+F 3 "~" H 3650 3200 50  0001 C CNN
+	1    3650 3200
+	-1   0    0    1
 $EndComp
 Wire Wire Line
-	3150 3200 2900 3200
-Wire Wire Line
-	3150 3300 2900 3300
+	3350 3300 3100 3300
 $Comp
 L power:+12V #PWR?
 U 1 1 60E4A1A7
-P 2900 3200
+P 3100 3300
 AR Path="/60E4A1A7" Ref="#PWR?"  Part="1"
 AR Path="/608889A3/60E4A1A7" Ref="#PWR0140"  Part="1"
-F 0 "#PWR0140" H 2900 3050 50  0001 C CNN
-F 1 "+12V" H 2915 3373 50  0000 C CNN
-F 2 "" H 2900 3200 50  0001 C CNN
-F 3 "" H 2900 3200 50  0001 C CNN
-	1    2900 3200
-	1    0    0    -1
+F 0 "#PWR0140" H 3100 3150 50  0001 C CNN
+F 1 "+12V" H 3115 3473 50  0000 C CNN
+F 2 "" H 3100 3300 50  0001 C CNN
+F 3 "" H 3100 3300 50  0001 C CNN
+	1    3100 3300
+	-1   0    0    1
 $EndComp
 $Comp
 L power:GND #PWR?
 U 1 1 60E4A59F
-P 2900 3300
+P 3100 3100
 AR Path="/60E4A59F" Ref="#PWR?"  Part="1"
 AR Path="/608889A3/60E4A59F" Ref="#PWR0142"  Part="1"
-F 0 "#PWR0142" H 2900 3050 50  0001 C CNN
-F 1 "GND" H 2905 3127 50  0000 C CNN
-F 2 "" H 2900 3300 50  0001 C CNN
-F 3 "" H 2900 3300 50  0001 C CNN
-	1    2900 3300
-	1    0    0    -1
+F 0 "#PWR0142" H 3100 2850 50  0001 C CNN
+F 1 "GND" H 3105 2927 50  0000 C CNN
+F 2 "" H 3100 3100 50  0001 C CNN
+F 3 "" H 3100 3100 50  0001 C CNN
+	1    3100 3100
+	-1   0    0    1
 $EndComp
 Wire Wire Line
@@
 Connection ~ 5000 2000
 NoConn ~ 4950 4250
+Wire Wire Line
+	3100 3100 3350 3100
 $EndSCHEMATC

Commit message: holes
Parts:
- Led1: renamed from LedRed1; value LED_Small -> LED_RED
Changed lines of the file:
@@
 	5200 4350 5200 4250
 $Comp
-L Device:LED_Small LedRed1
+L Device:LED_Small Led1
 U 1 1 6089055D
 P 5750 4850
-F 0 "LedRed1" V 5796 4780 50  0000 R CNN
-F 1 "LED_Small" V 5705 4780 50  0000 R CNN
+F 0 "Led1" V 5796 4780 50  0000 R CNN
+F 1 "LED_RED" V 5705 4780 50  0000 R CNN
 F 2 "LED_SMD:LED_0805_2012Metric" V 5750 4850 50  0001 C CNN
 F 3 "~" V 5750 4850 50  0001 C CNN
